Commit message: more notes on the cam instrisic

File: urdf/_d435_gazebo_config.xacro (robot description, xacro)
@@ -10,8 +10,28 @@
 <xacro:arg name="infra_res" default="640x480"/>
 <xacro:property name="INFRA_RES" value="$(arg infra_res)" />
-<xacro:if value="${COLOR_RES == '640x480'}">
+<xacro:if value="${COLOR_RES == '1920x1080'}">
+  <xacro:property name="color_width" value="1920"/>
+  <xacro:property name="color_height" value="1080"/>
+  <xacro:property name="color_fps" value="30"/> <!--6 15 30-->
+  <xacro:property name="color_fx" value="1364.58154296875"/>
+  <xacro:property name="color_fy" value="1364.4825439453125"/>
+  <xacro:property name="color_cx" value="974.0638427734375"/>
+  <xacro:property name="color_cy" value="572.7390747070312"/>
+</xacro:if>
+<xacro:if value="${COLOR_RES == '1280x720'}">
+  <xacro:property name="color_width" value="1280"/>
+  <xacro:property name="color_height" value="720"/>
+  <xacro:property name="color_fps" value="30"/> <!--6 15 30-->
+  <xacro:property name="color_fx" value="909.7210083007812"/>
+  <xacro:property name="color_fy" value="909.655029296875"/>
+  <xacro:property name="color_cx" value="649.3759155273438"/>
+  <xacro:property name="color_cy" value="381.8260498046875"/>
+</xacro:if>
+<xacro:if value="${COLOR_RES == '960x540'}"></xacro:if>
+<xacro:if value="${COLOR_RES == '848x480'}"></xacro:if>
+<xacro:if value="${COLOR_RES == '640x480'}"> <!--default roslaunch of real cam-->
   <xacro:property name="color_width" value="640"/>
   <xacro:property name="color_height" value="480"/>
-  <xacro:property name="color_fps" value="30"/>
+  <xacro:property name="color_fps" value="30"/> <!--6 15 30 60-->
   <xacro:property name="color_fx" value="606.4806518554688"/>
   <xacro:property name="color_fy" value="606.4366455078125"/>
@@ -19,30 +39,50 @@
   <xacro:property name="color_cy" value="254.5507049560547"/>
 </xacro:if>
-<xacro:if value="${COLOR_RES == '1280x720'}">
-  <xacro:property name="color_width" value="1280"/>
-  <xacro:property name="color_height" value="720"/>
-  <xacro:property name="color_fps" value="30"/>
-  <xacro:property name="color_fx" value="909.7210083007812"/>
-  <xacro:property name="color_fy" value="909.655029296875"/>
-  <xacro:property name="color_cx" value="649.3759155273438"/>
-  <xacro:property name="color_cy" value="381.8260498046875"/>
+<xacro:if value="${COLOR_RES == '640x360'}"></xacro:if>
+<xacro:if value="${COLOR_RES == '424x240'}"></xacro:if>
+<xacro:if value="${COLOR_RES == '320x240'}"></xacro:if>
+<xacro:if value="${COLOR_RES == '320x180'}"></xacro:if>
+<!-- NOTE: on real camera, for the aligned to color version the instrisic are the same of color one -->
+<xacro:if value="${DEPTH_RES == '1280x720'}">
+  <xacro:property name="depth_width" value="1280"/>
+  <xacro:property name="depth_height" value="720"/>
+  <xacro:property name="depth_fps" value="30"/> <!--  6 15 30 for this res -->
+  <xacro:property name="depth_fx" value="650.98046875"/>
+  <xacro:property name="depth_fy" value="650.98046875"/>
+  <xacro:property name="depth_cx" value="639.7286987304688"/>
+  <xacro:property name="depth_cy" value="361.9244384765625"/>
+  <xacro:property name="clip_distance_min" value="0.280"/>
 </xacro:if>
-<xacro:if value="${COLOR_RES == '1920x1080'}">
-  <xacro:property name="color_width" value="1920"/>
-  <xacro:property name="color_height" value="1080"/>
-  <xacro:property name="color_fps" value="30"/>
-  <xacro:property name="color_fx" value="1364.58154296875"/>
-  <xacro:property name="color_fy" value="1364.4825439453125"/>
-  <xacro:property name="color_cx" value="974.0638427734375"/>
-  <xacro:property name="color_cy" value="572.7390747070312"/>
-</xacro:if>
-<xacro:if value="${DEPTH_RES == '848x480'}">
+<xacro:if value="${DEPTH_RES == '848x480'}"> <!--default roslaunch of real cam-->
   <xacro:property name="depth_width" value="848"/>
   <xacro:property name="depth_height" value="480"/>
-  <xacro:property name="depth_fps" value="30"/>
+  <xacro:property name="depth_fps" value="30"/> <!-- 6 15 30 60 90 avaiable from this to lower res -->
   <xacro:property name="depth_fx" value="431.2745666503906"/>
   <xacro:property name="depth_fy" value="431.2745666503906"/>
   <xacro:property name="depth_cx" value="423.82025146484375"/>
   <xacro:property name="depth_cy" value="241.2349395751953"/>
+  <xacro:property name="clip_distance_min" value="0.195"/>
+</xacro:if>
+<xacro:if value="${DEPTH_RES == '640x480'}">
+  <xacro:property name="depth_width" value="640"/>
+  <xacro:property name="depth_height" value="480"/>
+  <xacro:property name="depth_fps" value="30"/> <!-- 6 15 30 60 90 avaiable from this to lower res -->
+  <xacro:property name="depth_fx" value="390.5882873535156"/>
+  <xacro:property name="depth_fy" value="390.5882873535156"/>
+  <xacro:property name="depth_cx" value="319.83721923828125"/>
+  <xacro:property name="depth_cy" value="241.14466857910156"/>
+  <xacro:property name="clip_distance_min" value="0.175"/>
+</xacro:if>
+<xacro:if value="${DEPTH_RES == '640x360'}"></xacro:if>
+<xacro:if value="${DEPTH_RES == '480x270'}"></xacro:if>
+<xacro:if value="${DEPTH_RES == '424x240'}">
+  <xacro:property name="depth_width" value="424"/>
+  <xacro:property name="depth_height" value="240"/>
+  <xacro:property name="depth_fps" value="30"/>
+  <xacro:property name="depth_fx" value="215.6372833251953"/>
+  <xacro:property name="depth_fy" value="215.6372833251953"/>
+  <xacro:property name="depth_cx" value="211.91012573242188"/>
+  <xacro:property name="depth_cy" value="120.63746643066406"/>
+  <xacro:property name="clip_distance_min" value="0.105"/>
 </xacro:if>
 <xacro:if value="${INFRA_RES == '640x480'}">
