Commit message: upd urdf/gazebo files to `realsense-ros/ros1-legacy` commit 9398c98

File: urdf/_d435.gazebo.xacro (robot description, xacro)
@@ -1,10 +1,10 @@
 <?xml version="1.0"?>
 <!--
-Aknolegment: This file was originally copied from the realsense repository of
+Acknolegment: This file was originally copied from the realsense repository of
 pal-robotics-forks( https://github.com/pal-robotics-forks/realsense/ )
 and then modified.
 License: Apache 2.0. See LICENSE file in root directory.
 Copyright(c) 2017 PAL Robotics, S.L. All Rights Reserved
-This is the Gazebo URDF model for the Intel RealSense D435 camera
+This is the Gazebo URDF model for the Intel RealSense D435/D435i camera
 -->
 <robot xmlns:xacro="http://ros.org/wiki/xacro">
@@ -16,4 +16,10 @@
                                           infrared1_optical_frame
                                           infrared2_optical_frame
+                                          accel_optical_frame
+                                          gyro_optical_frame
+                                          has_imu:=false
+                                          unite_imu_method:=false
+                                          accel_fps:=250
+                                          gyro_fps:=400
                                           clip_distance:=-1.0
                                           depth_width:=1280
@@ -153,4 +159,57 @@
         <visualize>false</visualize>
       </sensor>
+      <xacro:if value="${has_imu}">
+        <!-- IMU -->
+        <xacro:if value="${unite_imu_method == 'copy' or unite_imu_method == 'linear_interpolation'}">
+          <sensor name="${camera_name}imu" type="imu">
+            <always_on>true</always_on>
+            <update_rate>${gyro_fps}</update_rate>
+            <topic>${camera_name}/imu/sample</topic>
+            <plugin name="${camera_name}imu" filename="libgazebo_ros_imu_sensor.so">
+              <topicName>${camera_name}/imu/sample</topicName>
+              <bodyName>${camera_name}_link</bodyName>
+              <frameName>${gyro_optical_frame}</frameName>
+              <updateRateHZ>${gyro_fps}</updateRateHZ>
+              <gaussianNoise>0.1</gaussianNoise>
+              <xyzOffset>0 0 0</xyzOffset>
+              <rpyOffset>0 0 0</rpyOffset>
+            </plugin>
+          </sensor>
+        </xacro:if>
+        <!-- Accel and gyro -->
+        <xacro:unless value="${unite_imu_method == 'copy' or unite_imu_method == 'linear_interpolation'}">
+          <sensor name="${camera_name}accel" type="imu">
+            <always_on>true</always_on>
+            <update_rate>${accel_fps}</update_rate>
+            <topic>${camera_name}/accel/sample</topic>
+            <plugin name="${topics_ns}_accel_plugin" filename="librealsense_gazebo_accel_sensor.so">
+              <topicName>${camera_name}/accel/sample</topicName>
+              <bodyName>${camera_name}_link</bodyName>
+              <updateRateHZ>${accel_fps}</updateRateHZ>
+              <gaussianNoise>0.1</gaussianNoise>
+              <xyzOffset>0 0 0</xyzOffset>
+              <rpyOffset>0 0 0</rpyOffset>
+              <frameName>${accel_optical_frame}</frameName>
+              <initialOrientationAsReference>false</initialOrientationAsReference>
+            </plugin>
+            <pose>0 0 0 0 0 0</pose>
+          </sensor>
+          <sensor name="${camera_name}gyro" type="imu">
+            <always_on>true</always_on>
+            <update_rate>${gyro_fps}</update_rate>
+            <topic>${camera_name}/gyro/sample</topic>
+            <plugin name="${topics_ns}_gyro_plugin" filename="librealsense_gazebo_gyro_sensor.so">
+              <topicName>${camera_name}/gyro/sample</topicName>
+              <bodyName>${camera_name}_link</bodyName>
+              <updateRateHZ>${gyro_fps}</updateRateHZ>
+              <gaussianNoise>0.1</gaussianNoise>
+              <xyzOffset>0 0 0</xyzOffset>
+              <rpyOffset>0 0 0</rpyOffset>
+              <frameName>${gyro_optical_frame}</frameName>
+              <initialOrientationAsReference>false</initialOrientationAsReference>
+            </plugin>
+          </sensor>
+        </xacro:unless>
+      </xacro:if>
     </gazebo>
     <gazebo>

File: urdf/_d435.urdf.xacro (robot description, xacro)
@@ -1,20 +1,34 @@
 <?xml version="1.0"?>
 <!--
-Aknolegment: This file was copied from the realsense repository of
+Acknolegment: This file was copied from the realsense repository of
 pal-robotics-forks( https://github.com/pal-robotics-forks/realsense/ ).
 and then modified.
 License: Apache 2.0. See LICENSE file in root directory.
 Copyright(c) 2017 Intel Corporation. All Rights Reserved
-This is the URDF model for the Intel RealSense 430 camera, in it's
+This is the URDF model for the Intel RealSense 430 camera, in its
 aluminum peripherial evaluation case.
 -->
 <robot name="sensor_d435" xmlns:xacro="http://ros.org/wiki/xacro">
-  <!--File includes-->
+  <!-- Includes -->
+  <xacro:property name="realsense_materials_defined" default="false" />
+  <xacro:unless value="${realsense_materials_defined}">
+    <xacro:property name="realsense_materials_defined" value="true" />
+    <xacro:include filename="$(find realsense_gazebo_description)/urdf/_materials.urdf.xacro" />
+  </xacro:unless>
+  <xacro:include filename="$(find realsense_gazebo_description)/urdf/_usb_plug.urdf.xacro" />
   <xacro:include filename="$(find realsense_gazebo_description)/urdf/_d435.gazebo.xacro"/>
   <xacro:macro name="sensor_d435" params="parent
+                                          *origin
                                           name:=camera
+                                          use_nominal_extrinsics:=false
+                                          add_plug:=false
+                                          use_mesh:=true
                                           topics_ns:=camera
                                           align_depth:=false
                                           enable_pointCloud:=false
+                                          has_imu:=false
+                                          unite_imu_method:=false
+                                          accel_fps:=250
+                                          gyro_fps:=400
                                           clip_distance:=-1.0
                                           depth_width:=1280
@@ -27,11 +41,11 @@
                                           color_height:=1080
                                           color_fps:=30
-                                          visualize:=false
-                                          *origin">
+                                          visualize:=false">
+<!--  <xacro:property name="module" value="${xacro.load_yaml(filename)}"/> -->
     <xacro:property name="M_PI" value="3.1415926535897931"/>
     <!-- The following values are approximate, and the camera node
      publishing TF values with actual calibrated camera extrinsic values -->
-    <xacro:property name="d435_cam_depth_to_left_ir_offset" value="0.0"/>
-    <xacro:property name="d435_cam_depth_to_right_ir_offset" value="-0.050"/>
+    <xacro:property name="d435_cam_depth_to_infra1_offset" value="0.0"/>
+    <xacro:property name="d435_cam_depth_to_infra2_offset" value="-0.050"/>
     <xacro:property name="d435_cam_depth_to_color_offset" value="0.015"/>
     <!-- The following values model the aluminum peripherial case for the
@@ -42,4 +56,10 @@
     <xacro:property name="d435_cam_depth" value="0.02505"/>
     <xacro:property name="d435_cam_mount_from_center_offset" value="0.0149"/>
+    <!-- glass cover is 0.1 mm inwards from front aluminium plate -->
+    <xacro:property name="d435_glass_to_front" value="0.1e-3"/>
+    <!-- see datasheet Revision 007, Fig. 4-4 page 65 -->
+    <xacro:property name="d435_zero_depth_to_glass" value="4.2e-3"/>
+    <!-- convenience precomputation to avoid clutter-->
+    <xacro:property name="d435_mesh_x_offset" value="${d435_cam_mount_from_center_offset-d435_glass_to_front-d435_zero_depth_to_glass}"/>
     <!-- The following offset is relative the the physical D435 camera peripherial
   	camera tripod mount -->
@@ -47,7 +67,4 @@
     <xacro:property name="d435_cam_depth_py" value="0.0175"/>
     <xacro:property name="d435_cam_depth_pz" value="${d435_cam_height/2}"/>
-    <material name="${name}_aluminum">
-	  <color rgba="0.5 0.5 0.5 1"/>
-    </material>
     <!-- camera body, with origin at bottom screw mount -->
     <joint name="${name}_joint" type="fixed">
@@ -58,5 +75,5 @@
     <link name="${name}_bottom_screw_frame"/>
     <joint name="${name}_link_joint" type="fixed">
-      <origin xyz="0 ${d435_cam_depth_py} ${d435_cam_depth_pz}" rpy="0 0 0"/>
+      <origin xyz="${d435_mesh_x_offset} ${d435_cam_depth_py} ${d435_cam_depth_pz}" rpy="0 0 0"/>
       <parent link="${name}_bottom_screw_frame"/>
       <child link="${name}_link"/>
@@ -64,77 +81,92 @@
     <link name="${name}_link">
       <visual>
-      <origin xyz="${d435_cam_mount_from_center_offset} ${-d435_cam_depth_py} 0" rpy="${M_PI/2} 0 ${M_PI/2}"/>
-        <geometry>
-          <!-- <box size="${d435_cam_width} ${d435_cam_height} ${d435_cam_depth}"/> -->
-          <mesh filename="package://realsense2_description/meshes/d435.dae"/>
-          <!--<mesh filename="package://realsense2_description/meshes/d435/d435.dae"/>-->
-        </geometry>
-        <material name="${name}_aluminum"/>
+        <xacro:if value="${use_mesh}">
+          <!-- the mesh origin is at front plate in between the two infrared camera axes -->
+          <origin xyz="${d435_zero_depth_to_glass + d435_glass_to_front} ${-d435_cam_depth_py} 0" rpy="${M_PI/2} 0 ${M_PI/2}"/>
+          <geometry>
+            <mesh filename="package://realsense2_description/meshes/d435.dae" />
+          </geometry>
+        </xacro:if>
+        <xacro:unless value="${use_mesh}">
+          <origin xyz="0 ${-d435_cam_depth_py} 0" rpy="0 0 0"/>
+          <geometry>
+            <box size="${d435_cam_depth} ${d435_cam_width} ${d435_cam_height}"/>
+          </geometry>
+          <material name="aluminum"/>
+        </xacro:unless>
       </visual>
       <collision>
         <origin xyz="0 ${-d435_cam_depth_py} 0" rpy="0 0 0"/>
         <geometry>
-        <box size="${d435_cam_depth} ${d435_cam_width} ${d435_cam_height}"/>
+          <box size="${d435_cam_depth} ${d435_cam_width} ${d435_cam_height}"/>
         </geometry>
       </collision>
       <inertial>
         <!-- The following are not reliable values, and should not be used for modeling -->
-        <mass value="0.564"/>
-        <origin xyz="0 0 0"/>
-        <inertia ixx="0.003881243" ixy="0.0" ixz="0.0" iyy="0.000498940" iyz="0.0" izz="0.003879257"/>
+        <mass value="0.072" />
+        <origin xyz="0 0 0" />
+        <inertia ixx="0.003881243" ixy="0.0" ixz="0.0" iyy="0.000498940" iyz="0.0" izz="0.003879257" />
       </inertial>
     </link>
-    <!-- camera depth joints and links -->
-    <joint name="${name}_depth_joint" type="fixed">
-      <origin xyz="0 0 0" rpy="0 0 0"/>
-      <parent link="${name}_link"/>
-      <child link="${name}_depth_frame"/>
-    </joint>
-    <link name="${name}_depth_frame"/>
-    <joint name="${name}_depth_optical_joint" type="fixed">
-      <origin xyz="0 0 0" rpy="${-M_PI/2} 0 ${-M_PI/2}"/>
-      <parent link="${name}_depth_frame"/>
-      <child link="${name}_depth_optical_frame"/>
-    </joint>
-    <link name="${name}_depth_optical_frame"/>
-    <!-- camera left IR joints and links -->
-    <joint name="${name}_left_ir_joint" type="fixed">
-      <origin xyz="0 ${d435_cam_depth_to_left_ir_offset} 0" rpy="0 0 0"/>
-      <parent link="${name}_depth_frame"/>
-      <child link="${name}_left_ir_frame"/>
-    </joint>
-    <link name="${name}_left_ir_frame"/>
-    <joint name="${name}_left_ir_optical_joint" type="fixed">
-      <origin xyz="0 0 0" rpy="${-M_PI/2} 0 ${-M_PI/2}"/>
-      <parent link="${name}_left_ir_frame"/>
-      <child link="${name}_left_ir_optical_frame"/>
-    </joint>
-    <link name="${name}_left_ir_optical_frame"/>
-    <!-- camera right IR joints and links -->
-    <joint name="${name}_right_ir_joint" type="fixed">
-      <origin xyz="0 ${d435_cam_depth_to_right_ir_offset} 0" rpy="0 0 0"/>
-      <parent link="${name}_depth_frame"/>
-      <child link="${name}_right_ir_frame"/>
-    </joint>
-    <link name="${name}_right_ir_frame"/>
-    <joint name="${name}_right_ir_optical_joint" type="fixed">
-      <origin xyz="0 0 0" rpy="${-M_PI/2} 0 ${-M_PI/2}"/>
-      <parent link="${name}_right_ir_frame"/>
-      <child link="${name}_right_ir_optical_frame"/>
-    </joint>
-    <link name="${name}_right_ir_optical_frame"/>
-    <!-- camera color joints and links -->
-    <joint name="${name}_color_joint" type="fixed">
-      <origin xyz="0 ${d435_cam_depth_to_color_offset} 0" rpy="0 0 0"/>
-      <parent link="${name}_depth_frame"/>
-      <child link="${name}_color_frame"/>
-    </joint>
-    <link name="${name}_color_frame"/>
-    <joint name="${name}_color_optical_joint" type="fixed">
-      <origin xyz="0 0 0" rpy="${-M_PI/2} 0 ${-M_PI/2}"/>
-      <parent link="${name}_color_frame"/>
-      <child link="${name}_color_optical_frame"/>
-    </joint>
-    <link name="${name}_color_optical_frame"/>
+    <!-- Use the nominal extrinsics between camera frames if the calibrated extrinsics aren't being published. e.g. running the device in simulation  -->
+    <xacro:if value="${use_nominal_extrinsics}">
+      <!-- camera depth joints and links -->
+      <joint name="${name}_depth_joint" type="fixed">
+        <origin xyz="0 0 0" rpy="0 0 0"/>
+        <parent link="${name}_link"/>
+        <child link="${name}_depth_frame" />
+      </joint>
+      <link name="${name}_depth_frame"/>
+      <joint name="${name}_depth_optical_joint" type="fixed">
+        <origin xyz="0 0 0" rpy="${-M_PI/2} 0 ${-M_PI/2}" />
+        <parent link="${name}_depth_frame" />
+        <child link="${name}_depth_optical_frame" />
+      </joint>
+      <link name="${name}_depth_optical_frame"/>
+      <!-- camera left IR joints and links -->
+      <joint name="${name}_infra1_joint" type="fixed">
+        <origin xyz="0 ${d435_cam_depth_to_infra1_offset} 0" rpy="0 0 0" />
+        <parent link="${name}_link" />
+        <child link="${name}_infra1_frame" />
+      </joint>
+      <link name="${name}_infra1_frame"/>
+      <joint name="${name}_infra1_optical_joint" type="fixed">
+        <origin xyz="0 0 0" rpy="${-M_PI/2} 0 ${-M_PI/2}" />
+        <parent link="${name}_infra1_frame" />
+        <child link="${name}_infra1_optical_frame" />
+      </joint>
+      <link name="${name}_infra1_optical_frame"/>
+      <!-- camera right IR joints and links -->
+      <joint name="${name}_infra2_joint" type="fixed">
+        <origin xyz="0 ${d435_cam_depth_to_infra2_offset} 0" rpy="0 0 0" />
+        <parent link="${name}_link" />
+        <child link="${name}_infra2_frame" />
+      </joint>
+      <link name="${name}_infra2_frame"/>
+      <joint name="${name}_infra2_optical_joint" type="fixed">
+        <origin xyz="0 0 0" rpy="${-M_PI/2} 0 ${-M_PI/2}" />
+        <parent link="${name}_infra2_frame" />
+        <child link="${name}_infra2_optical_frame" />
+      </joint>
+      <link name="${name}_infra2_optical_frame"/>
+      <!-- camera color joints and links -->
+      <joint name="${name}_color_joint" type="fixed">
+        <origin xyz="0 ${d435_cam_depth_to_color_offset} 0" rpy="0 0 0" />
+        <parent link="${name}_link" />
+        <child link="${name}_color_frame" />
+      </joint>
+      <link name="${name}_color_frame"/>
+      <joint name="${name}_color_optical_joint" type="fixed">
+        <origin xyz="0 0 0" rpy="${-M_PI/2} 0 ${-M_PI/2}" />
+        <parent link="${name}_color_frame" />
+        <child link="${name}_color_optical_frame" />
+      </joint>
+      <link name="${name}_color_optical_frame"/>
+    </xacro:if>
+    <xacro:if value="${add_plug}">
+      <xacro:usb_plug parent="${name}_link" name="${name}_usb_plug">
+        <origin xyz="${d435_cam_mount_from_center_offset - 0.02095} ${-d435_cam_depth_py - 0.0353} 0" rpy="0 0 0"/>
+      </xacro:usb_plug>
+    </xacro:if>
     <!-- Realsense Gazebo Plugin -->
     <xacro:gazebo_d435  camera_name="${name}"
@@ -149,10 +181,16 @@
                         color_height="${color_height}"
                         color_fps="${color_fps}"
-                        infrared1_optical_frame="${name}_left_ir_optical_frame"
-                        infrared2_optical_frame="${name}_right_ir_optical_frame"
+                        infrared1_optical_frame="${name}_infra1_optical_frame"
+                        infrared2_optical_frame="${name}_infra2_optical_frame"
                         infra_width="${infra_width}"
                         infra_height="${infra_height}"
                         infra_fps="${infra_fps}"
+                        has_imu="${has_imu}"
+                        accel_optical_frame="${name}_accel_optical_frame"
+                        gyro_optical_frame="${name}_gyro_optical_frame"
+                        accel_fps="${accel_fps}"
+                        gyro_fps="${gyro_fps}"
                         enable_pointCloud="${enable_pointCloud}"
+                        unite_imu_method="${unite_imu_method}"
                         clip_distance="${clip_distance}"
                         align_depth="${align_depth}"
