Commit message: (feat) Added gazebo xacro to insert camera and depth camera. The option 'align_depth' allows to create the depth camera with same spec as the color one in the color_frame so that it mimics the behavior of the realsense.
(feat) Created basic world file in'worlds' to allow the usage of the sensor plugin in gazebo (necessary to load the sensors in the simulation.

(refactor) Updated launch file to not use the Tf publisher since the pose is alredy passed to the URDF via parameter and added Gazebo Harmonic bridges to republish the topics in ROS2.

File: urdf/_d435i.gazebo.xacro (robot description, xacro)
@@ -21,4 +21,5 @@
                                           depth_cx:= 423.82025146484375
                                           depth_cy:= 241.2349395751953
+                                          infra_enable:=false
                                           infra_width:=640
                                           infra_height:=480
@@ -47,4 +48,5 @@
     <!-- Load parameters to model's main link-->
     <xacro:property name="deg_to_rad" value="0.01745329251994329577" />
+    <xacro:property name="INFRARED" value="${infra_enable}" />
     <gazebo reference="${reference_link}">
       <self_collide>0</self_collide>
@@ -62,6 +64,6 @@
       <min_depth>0</min_depth>-->
       <sensor name="${camera_name}_color" type="camera">
-        <gz_frame_id>${camera_name}/camera_color_optical_frame</gz_frame_id>
-        <optical_frame_id>${camera_name}/camera_color_optical_frame</optical_frame_id>
+        <gz_frame_id>${camera_name}_color_frame</gz_frame_id>
+        <optical_frame_id>${camera_name}_color_optical_frame</optical_frame_id>
         <topic>${camera_name}/color/image_raw</topic>
         <camera name="${camera_name}">
@@ -77,9 +79,9 @@
             <far>100</far>
           </clip>
-          <noise>
+          <!-- <noise>
             <type>gaussian</type>
             <mean>0.0</mean>
             <stddev>0.007</stddev>
-          </noise>
+          </noise> -->
           <lens>
             <projection>
@@ -104,91 +106,99 @@
         <visualize>${visualize}</visualize>
       </sensor>
-      <sensor name="${camera_name}ired1" type="camera">
-        <camera name="${camera_name}">
-          <horizontal_fov>${85.2*deg_to_rad}</horizontal_fov>
-          <image>
-            <width>${infra_width}</width>
-            <height>${infra_height}</height>
-            <format>L_INT8</format>
-          </image>
-          <clip>
-            <near>0.1</near>
-            <far>100</far>
-          </clip>
-          <noise>
-            <type>gaussian</type>
-            <mean>0.0</mean>
-            <stddev>0.05</stddev>
-          </noise>
-          <lens>
-            <projection>
-              <p_fx>${infra_fx}</p_fx>
-              <p_fy>${infra_fy}</p_fy>
-              <p_cx>${infra_cx}</p_cx>
-              <p_cy>${infra_cy}</p_cy>
-              <tx>0</tx>
-              <ty>0</ty>
-            </projection>
-            <intrinsics>
-              <fx>${infra_fx}</fx>
-              <fy>${infra_fy}</fy>
-              <cx>${infra_cx}</cx>
-              <cy>${infra_cy}</cy>
-              <s>0</s>
-            </intrinsics>
-          </lens>
-        </camera>
-        <always_on>1</always_on>
-        <update_rate>${infra_fps}</update_rate>
-        <visualize>false</visualize>
-      </sensor>
-      <sensor name="${camera_name}ired2" type="camera">
-        <camera name="${camera_name}">
-          <horizontal_fov>${85.2*deg_to_rad}</horizontal_fov>
-          <image>
-            <width>${infra_width}</width>
-            <height>${infra_height}</height>
-            <format>L_INT8</format>
-          </image>
-          <clip>
-            <near>0.1</near>
-            <far>100</far>
-          </clip>
-          <noise>
-            <type>gaussian</type>
-            <mean>0.0</mean>
-            <stddev>0.05</stddev>
-          </noise>
-          <lens>
-            <projection>
-              <p_fx>${infra_fx}</p_fx>
-              <p_fy>${infra_fy}</p_fy>
-              <p_cx>${infra_cx}</p_cx>
-              <p_cy>${infra_cy}</p_cy>
-              <tx>${infra2_tx}</tx>
-              <ty>0</ty>
-            </projection>
-            <intrinsics>
-              <fx>${infra_fx}</fx>
-              <fy>${infra_fy}</fy>
-              <cx>${infra_cx}</cx>
-              <cy>${infra_cy}</cy>
-              <s>0</s>
-            </intrinsics>
-          </lens>
-        </camera>
-        <always_on>1</always_on>
-        <update_rate>${infra_fps}</update_rate>
-        <visualize>false</visualize>
-      </sensor>
+      <xacro:if value="${INFRARED}">
+        <sensor name="${camera_name}_ired1" type="camera">
+          <gz_frame_id>${camera_name}_infra1_frame</gz_frame_id>
+          <optical_frame_id>${camera_name}_infra1_optical_frame</optical_frame_id>
+          <topic>${camera_name}/infra1/image_raw</topic>
+          <camera name="${camera_name}_ired1">
+            <horizontal_fov>${85.2*deg_to_rad}</horizontal_fov>
+            <image>
+              <width>${infra_width}</width>
+              <height>${infra_height}</height>
+              <format>L_INT8</format>
+            </image>
+            <clip>
+              <near>0.1</near>
+              <far>100</far>
+            </clip>
+            <!-- <noise>
+              <type>gaussian</type>
+              <mean>0.0</mean>
+              <stddev>0.05</stddev>
+            </noise> -->
+            <lens>
+              <projection>
+                <p_fx>${infra_fx}</p_fx>
+                <p_fy>${infra_fy}</p_fy>
+                <p_cx>${infra_cx}</p_cx>
+                <p_cy>${infra_cy}</p_cy>
+                <tx>0</tx>
+                <ty>0</ty>
+              </projection>
+              <intrinsics>
+                <fx>${infra_fx}</fx>
+                <fy>${infra_fy}</fy>
+                <cx>${infra_cx}</cx>
+                <cy>${infra_cy}</cy>
+                <s>0</s>
+              </intrinsics>
+            </lens>
+          </camera>
+          <always_on>1</always_on>
+          <update_rate>${infra_fps}</update_rate>
+          <visualize>false</visualize>
+        </sensor>
+        <sensor name="${camera_name}_ired2" type="camera">
+          <gz_frame_id>${camera_name}_infra2_frame</gz_frame_id>
+          <optical_frame_id>${camera_name}_infra2_optical_frame</optical_frame_id>
+          <topic>${camera_name}/infra2/image_raw</topic>
+          <camera name="${camera_name}_ired2">
+            <horizontal_fov>${85.2*deg_to_rad}</horizontal_fov>
+            <image>
+              <width>${infra_width}</width>
+              <height>${infra_height}</height>
+              <format>L_INT8</format>
+            </image>
+            <clip>
+              <near>0.1</near>
+              <far>100</far>
+            </clip>
+            <!-- <noise>
+              <type>gaussian</type>
+              <mean>0.0</mean>
+              <stddev>0.05</stddev>
+            </noise> -->
+            <lens>
+              <projection>
+                <p_fx>${infra_fx}</p_fx>
+                <p_fy>${infra_fy}</p_fy>
+                <p_cx>${infra_cx}</p_cx>
+                <p_cy>${infra_cy}</p_cy>
+                <tx>${infra2_tx}</tx>
+                <ty>0</ty>
+              </projection>
+              <intrinsics>
+                <fx>${infra_fx}</fx>
+                <fy>${infra_fy}</fy>
+                <cx>${infra_cx}</cx>
+                <cy>${infra_cy}</cy>
+                <s>0</s>
+              </intrinsics>
+            </lens>
+          </camera>
+          <always_on>1</always_on>
+          <update_rate>${infra_fps}</update_rate>
+          <visualize>false</visualize>
+        </sensor>
+      </xacro:if>
       <sensor name="${camera_name}_depth" type="depth">
         <xacro:unless value="${align_depth}">
-          <gz_frame_id>${camera_name}/camera_depth_optical_frame</gz_frame_id>
-          <optical_frame_id>${camera_name}/camera_depth_optical_frame</optical_frame_id>
+          <gz_frame_id>${camera_name}_depth_frame</gz_frame_id>
+          <optical_frame_id>${camera_name}_depth_optical_frame</optical_frame_id>
           <topic>${camera_name}/depth/image_raw</topic>
         </xacro:unless>
         <xacro:if value="${align_depth}">
-          <gz_frame_id>${camera_name}/camera_color_optical_frame</gz_frame_id>
-          <optical_frame_id>${camera_name}/camera_color_optical_frame</optical_frame_id>
+          <gz_frame_id>${camera_name}_color_frame</gz_frame_id>
+          <optical_frame_id>${camera_name}_color_optical_frame</optical_frame_id>
           <topic>${camera_name}/aligned_depth_to_color/image_raw</topic>
         </xacro:if>
@@ -196,7 +206,7 @@
           <!-- align-depth settings -->
           <xacro:unless value="${align_depth}">
-            <camera_info_topic>${camera_name}/depth/camera_info</camera_info_topic>
-            <horizontal_fov>${85.2*deg_to_rad}</horizontal_fov>
-            <image>
+          <camera_info_topic>${camera_name}/depth/camera_info</camera_info_topic>
+          <horizontal_fov>${85.2*deg_to_rad}</horizontal_fov>
+          <image>
               <width>${depth_width}</width>
               <height>${depth_height}</height>
@@ -220,9 +230,9 @@
             </xacro:if>
           </clip>
-          <noise>
+          <!-- <noise>
             <type>gaussian</type>
             <mean>0.0</mean>
             <stddev>0.100</stddev>
-          </noise>
+          </noise> -->
           <lens>
             <xacro:unless value="${align_depth}">

File: urdf/_d435i.urdf.xacro (robot description, xacro)
@@ -23,4 +23,5 @@
   <xacro:include filename="$(find realsense_gazebo_description)/urdf/_materials.urdf.xacro" />
   <xacro:include filename="$(find realsense_gazebo_description)/urdf/_usb_plug.urdf.xacro" />
+  <xacro:include filename="$(find realsense_gazebo_description)/urdf/_d435i.gazebo.xacro" />
   <xacro:macro name="sensor_d435i" params="parent
                                           name:=camera
@@ -30,4 +31,5 @@
                                           publish_pointcloud:=false
                                           align_depth:=true
+                                          gazebo_urdf:=false
                                           clip_distance:=-1.0
                                           clip_distance_min:=0.195
@@ -39,4 +41,5 @@
                                           depth_cx:= 423.82025146484375
                                           depth_cy:= 241.2349395751953
+                                          infra_enable:=false
                                           infra_width:=640
                                           infra_height:=480
@@ -55,6 +58,11 @@
                                           color_cy:= 254.5507049560547
                                           visualize:=false
+                                          unite_imu_method:=false
+                                          accel_fps:=250
+                                          gyro_fps:=400
                                           *origin">
     <xacro:property name="M_PI" value="3.1415926535897931" />
+    <xacro:property name= "GAZEBO_URDF" value="${gazebo_urdf}" /> <!-- set true to load gazebo plugins -->
+    <xacro:property name="INFRARED" value="${infra_enable}" /> <!-- Set true to enable infrared sensors-->
     <!-- The following values are approximate, and the camera node
      publishing TF values with actual calibrated camera extrinsic values -->
@@ -137,29 +145,31 @@
       <link name="${name}_depth_optical_frame"/>
       <!-- camera left IR joints and links -->
-      <joint name="${name}_infra1_joint" type="fixed">
-        <origin xyz="0 ${d435_cam_depth_to_infra1_offset} 0" rpy="0 0 0" />
-        <parent link="${name}_link" />
-        <child link="${name}_infra1_frame" />
-      </joint>
-      <link name="${name}_infra1_frame"/>
-      <joint name="${name}_infra1_optical_joint" type="fixed">
-        <origin xyz="0 0 0" rpy="${-M_PI/2} 0 ${-M_PI/2}" />
-        <parent link="${name}_infra1_frame" />
-        <child link="${name}_infra1_optical_frame" />
-      </joint>
-      <link name="${name}_infra1_optical_frame"/>
-      <!-- camera right IR joints and links -->
-      <joint name="${name}_infra2_joint" type="fixed">
-        <origin xyz="0 ${d435_cam_depth_to_infra2_offset} 0" rpy="0 0 0" />
-        <parent link="${name}_link" />
-        <child link="${name}_infra2_frame" />
-      </joint>
-      <link name="${name}_infra2_frame"/>
-      <joint name="${name}_infra2_optical_joint" type="fixed">
-        <origin xyz="0 0 0" rpy="${-M_PI/2} 0 ${-M_PI/2}" />
-        <parent link="${name}_infra2_frame" />
-        <child link="${name}_infra2_optical_frame" />
-      </joint>
-      <link name="${name}_infra2_optical_frame"/>
+      <xacro:if value="${INFRARED}">
+        <joint name="${name}_infra1_joint" type="fixed">
+          <origin xyz="0 ${d435_cam_depth_to_infra1_offset} 0" rpy="0 0 0" />
+          <parent link="${name}_link" />
+          <child link="${name}_infra1_frame" />
+        </joint>
+        <link name="${name}_infra1_frame"/>
+        <joint name="${name}_infra1_optical_joint" type="fixed">
+          <origin xyz="0 0 0" rpy="${-M_PI/2} 0 ${-M_PI/2}" />
+          <parent link="${name}_infra1_frame" />
+          <child link="${name}_infra1_optical_frame" />
+        </joint>
+        <link name="${name}_infra1_optical_frame"/>
+        <!-- camera right IR joints and links -->
+        <joint name="${name}_infra2_joint" type="fixed">
+          <origin xyz="0 ${d435_cam_depth_to_infra2_offset} 0" rpy="0 0 0" />
+          <parent link="${name}_link" />
+          <child link="${name}_infra2_frame" />
+        </joint>
+        <link name="${name}_infra2_frame"/>
+        <joint name="${name}_infra2_optical_joint" type="fixed">
+          <origin xyz="0 0 0" rpy="${-M_PI/2} 0 ${-M_PI/2}" />
+          <parent link="${name}_infra2_frame" />
+          <child link="${name}_infra2_optical_frame" />
+        </joint>
+        <link name="${name}_infra2_optical_frame"/>
+      </xacro:if>
       <!-- camera color joints and links -->
       <joint name="${name}_color_joint" type="fixed">
@@ -207,4 +217,47 @@
       </xacro:usb_plug>
     </xacro:if>
+    <xacro:if value="${GAZEBO_URDF}">
+      <!-- Realsense Gazebo Plugin -->
+      <xacro:gazebo_d435i camera_name="${name}"
+                      reference_link="${name}_link"
+                      depth_optical_frame="${name}_depth_optical_frame"
+                      depth_width="${depth_width}"
+                      depth_height="${depth_height}"
+                      depth_fps="${depth_fps}"
+                      depth_fx="${depth_fx}"
+                      depth_fy="${depth_fy}"
+                      depth_cx="${depth_cx}"
+                      depth_cy="${depth_cy}"
+                      color_optical_frame="${name}_color_optical_frame"
+                      color_width="${color_width}"
+                      color_height="${color_height}"
+                      color_fps="${color_fps}"
+                      color_fx="${color_fx}"
+                      color_fy="${color_fy}"
+                      color_cx="${color_cx}"
+                      color_cy="${color_cy}"
+                      infrared1_optical_frame="${name}_infra1_ir_optical_frame"
+                      infrared2_optical_frame="${name}_infra2_ir_optical_frame"
+                      infra_enable="${infra_enable}"
+                      infra_width="${infra_width}"
+                      infra_height="${infra_height}"
+                      infra_fps="${infra_fps}"
+                      infra_fx="${infra_fx}"
+                      infra_fy="${infra_fy}"
+                      infra_cx="${infra_cx}"
+                      infra_cy="${infra_cy}"
+                      infra2_tx="${infra2_tx}"
+                      publish_pointcloud="${publish_pointcloud}"
+                      clip_distance="${clip_distance}"
+                      clip_distance_min="${clip_distance_min}"
+                      align_depth="${align_depth}"
+                      visualize="${visualize}"
+                      accel_optical_frame="${name}_accel_optical_frame"
+                      gyro_optical_frame="${name}_gyro_optical_frame"
+                      accel_fps="${accel_fps}"
+                      gyro_fps="${gyro_fps}"
+                      unite_imu_method="${unite_imu_method}"
+    />
+    </xacro:if>
   </xacro:macro>
 </robot>

File: urdf/d435_standalone.urdf.xacro (robot description, xacro)
@@ -14,9 +14,11 @@
     <xacro:arg name="add_plug" default="false" />
     <xacro:arg name="use_mesh" default="true" />
+    <xacro:arg name="gazebo_urdf" default="false" />
+    <xacro:arg name="infra_enable" default="false"/>
 	<xacro:include filename="$(find realsense_gazebo_description)/urdf/_d435.urdf.xacro"/>
  	<link name="$(arg parent)"/>
 	<xacro:sensor_d435 parent="$(arg parent)" name="$(arg name)"
         use_nominal_extrinsics="$(arg use_nominal_extrinsics)" add_plug="$(arg add_plug)"
-        use_mesh="$(arg use_mesh)"
+        use_mesh="$(arg use_mesh)" gazebo_urdf="$(arg gazebo_urdf)" infra_enable="$(arg infra_enable)"
         publish_pointcloud="$(arg publish_pointcloud)" align_depth="$(arg align_depth)">
 		<origin xyz="$(arg x) $(arg y) $(arg z)" rpy="$(arg roll) $(arg pitch) $(arg yaw)"/>

File: urdf/d435i_standalone.urdf.xacro (robot description, xacro)
@@ -14,9 +14,10 @@
     <xacro:arg name="add_plug" default="false" />
     <xacro:arg name="use_mesh" default="true" />
+    <xacro:arg name="gazebo_urdf" default="false" />
 	<xacro:include filename="$(find realsense_gazebo_description)/urdf/_d435i.urdf.xacro"/>
  	<link name="$(arg parent)"/>
 	<xacro:sensor_d435i parent="$(arg parent)" name="$(arg name)"
         use_nominal_extrinsics="$(arg use_nominal_extrinsics)" add_plug="$(arg add_plug)"
-        use_mesh="$(arg use_mesh)"
+        use_mesh="$(arg use_mesh)" gazebo_urdf="$(arg gazebo_urdf)"
         publish_pointcloud="$(arg publish_pointcloud)" align_depth="$(arg align_depth)">
 		<origin xyz="$(arg x) $(arg y) $(arg z)" rpy="$(arg roll) $(arg pitch) $(arg yaw)"/>
