Commit message: Added adaptive intrinsic based on image resolution like in the real camera
Updated mesh and material to visualize the model properly

File: urdf/_d435.gazebo.xacro (robot description, xacro)
@@ -6,6 +6,10 @@
 -->
 <robot xmlns:xacro="http://ros.org/wiki/xacro">
-  <xacro:macro name="gazebo_d435" params="reference_link
+  <xacro:macro name="gazebo_d435" params="
                                           camera_name:=camera
+                                          color_frame
+                                          depth_frame
+                                          infrared1_frame
+                                          infrared2_frame
                                           depth_optical_frame
                                           color_optical_frame
@@ -21,5 +25,5 @@
                                           depth_cx:= 423.82025146484375
                                           depth_cy:= 241.2349395751953
-                                          infra_enable:=false
+                                          enable_infrared:=false
                                           infra_width:=640
                                           infra_height:=480
@@ -38,11 +42,11 @@
                                           color_cy:= 254.5507049560547
                                           align_depth:=false
-                                          publish_pointcloud:=true
                                           visualize:=false
                                           ">
     <!-- Load parameters to model's main link-->
     <xacro:property name="deg_to_rad" value="0.01745329251994329577" />
-    <xacro:property name="INFRARED" value="${infra_enable}" />
-    <gazebo reference="${reference_link}">
+    <xacro:property name="INFRARED" value="${enable_infrared}" />
+    <!-- COLOR CAMERA -->
+    <gazebo reference="${color_frame}">
       <self_collide>0</self_collide>
       <enable_wind>0</enable_wind>
@@ -59,9 +63,9 @@
       <min_depth>0</min_depth>-->
       <sensor name="${camera_name}_color" type="camera">
-        <gz_frame_id>${camera_name}_color_frame</gz_frame_id>
-        <optical_frame_id>${camera_name}_color_optical_frame</optical_frame_id>
+        <gz_frame_id>${color_frame}</gz_frame_id>
         <topic>${camera_name}/color/image_raw</topic>
         <camera name="${camera_name}">
           <camera_info_topic>${camera_name}/color/camera_info</camera_info_topic>
+          <optical_frame_id>${color_optical_frame}</optical_frame_id>
           <horizontal_fov>${69.4*deg_to_rad}</horizontal_fov>
           <image>
@@ -74,9 +78,9 @@
             <far>100</far>
           </clip>
-          <noise>
+          <!-- <noise>
             <type>gaussian</type>
             <mean>0.0</mean>
             <stddev>0.007</stddev>
-          </noise>
+          </noise> -->
           <lens>
             <projection>
@@ -101,10 +105,13 @@
         <visualize>${visualize}</visualize>
       </sensor>
-      <xacro:if value="${INFRARED}">
+    </gazebo>
+    <!-- INFRARED -->
+    <xacro:if value="${INFRARED}">
+      <gazebo reference="${infrared1_frame}">
         <sensor name="${camera_name}_ired1" type="camera">
-          <gz_frame_id>${camera_name}_infra1_frame</gz_frame_id>
-          <optical_frame_id>${camera_name}_infra1_optical_frame</optical_frame_id>
+          <gz_frame_id>${infrared1_frame}</gz_frame_id>
           <topic>${camera_name}/infra1/image_raw</topic>
           <camera name="${camera_name}_ired1">
+            <optical_frame_id>${infrared1_optical_frame}</optical_frame_id>
             <horizontal_fov>${85.2*deg_to_rad}</horizontal_fov>
             <image>
@@ -144,9 +151,11 @@
           <visualize>false</visualize>
         </sensor>
+      </gazebo>
+      <gazebo reference="${infrared2_frame}">
         <sensor name="${camera_name}_ired2" type="camera">
-          <gz_frame_id>${camera_name}_infra2_frame</gz_frame_id>
-          <optical_frame_id>${camera_name}_infra2_optical_frame</optical_frame_id>
+          <gz_frame_id>${infrared1_frame}</gz_frame_id>
           <topic>${camera_name}/infra2/image_raw</topic>
           <camera name="${camera_name}_ired2">
+            <optical_frame_id>${infrared2_optical_frame}</optical_frame_id>
             <horizontal_fov>${85.2*deg_to_rad}</horizontal_fov>
             <image>
@@ -186,50 +195,91 @@
           <visualize>false</visualize>
         </sensor>
-      </xacro:if>
-      <sensor name="${camera_name}_depth" type="depth">
-        <xacro:unless value="${align_depth}">
-          <gz_frame_id>${camera_name}_depth_frame</gz_frame_id>
-          <optical_frame_id>${camera_name}_depth_optical_frame</optical_frame_id>
-          <topic>${camera_name}/depth/image_raw</topic>
-        </xacro:unless>
-        <xacro:if value="${align_depth}">
-          <gz_frame_id>${camera_name}_color_frame</gz_frame_id>
-          <optical_frame_id>${camera_name}_color_optical_frame</optical_frame_id>
+      </gazebo>
+    </xacro:if>
+    <!-- DEPTH CAMERA ALIGNED -->
+    <xacro:if value="${align_depth}">
+      <gazebo reference="${color_frame}">
+        <self_collide>0</self_collide>
+        <enable_wind>0</enable_wind>
+        <kinematic>0</kinematic>
+        <mu2>1</mu2>
+        <fdir1>0 0 0</fdir1>
+        <kp>1e+13</kp>
+        <kd>1</kd>
+        <sensor name="${camera_name}_depth" type="depth">
           <topic>${camera_name}/aligned_depth_to_color/image_raw</topic>
-        </xacro:if>
-        <camera name="${camera_name}">
-          <!-- align-depth settings -->
-          <xacro:unless value="${align_depth}">
-          <camera_info_topic>${camera_name}/depth/camera_info</camera_info_topic>
-          <horizontal_fov>${85.2*deg_to_rad}</horizontal_fov>
-          <image>
-              <width>${depth_width}</width>
-              <height>${depth_height}</height>
-            </image>
-          </xacro:unless>
-          <xacro:if value="${align_depth}">
+          <gz_frame_id>${color_frame}</gz_frame_id>
+          <camera name="${camera_name}_aligned_depth_camera">
             <camera_info_topic>${camera_name}/aligned_depth_to_color/camera_info</camera_info_topic>
+            <optical_frame_id>${color_optical_frame}</optical_frame_id>
             <horizontal_fov>${69.4*deg_to_rad}</horizontal_fov>
             <image>
               <width>${color_width}</width>
               <height>${color_height}</height>
-          </image>
-          </xacro:if>
-          <clip>
-            <near>${clip_distance_min}</near>
-            <xacro:unless value="${clip_distance > 0.0}">
-              <far>10</far>
-            </xacro:unless>
-            <xacro:if value="${clip_distance > 0.0}">
-              <far>${clip_distance}</far>
-            </xacro:if>
-          </clip>
-          <noise>
-            <type>gaussian</type>
-            <mean>0.0</mean>
-            <stddev>0.020</stddev>
-          </noise>
-          <lens>
-            <xacro:unless value="${align_depth}">
+            </image>
+            <clip>
+              <near>${clip_distance_min}</near>
+              <xacro:unless value="${clip_distance > 0.0}">
+                <far>10</far>
+              </xacro:unless>
+              <xacro:if value="${clip_distance > 0.0}">
+                <far>${clip_distance}</far>
+              </xacro:if>
+            </clip>
+            <lens>
+              <projection>
+                <p_fx>${color_fx}</p_fx>
+                <p_fy>${color_fy}</p_fy>
+                <p_cx>${color_cx}</p_cx>
+                <p_cy>${color_cy}</p_cy>
+                <tx>0</tx>
+                <ty>0</ty>
+              </projection>
+              <intrinsics>
+                <fx>${color_fx}</fx>
+                <fy>${color_fy}</fy>
+                <cx>${color_cx}</cx>
+                <cy>${color_cy}</cy>
+                <s>0</s>
+              </intrinsics>
+            </lens>
+          </camera>
+          <always_on>1</always_on>
+          <update_rate>${color_fps}</update_rate>
+          <visualize>false</visualize>
+        </sensor>
+      </gazebo>
+    </xacro:if>
+    <!-- DEPTH CAMERA NOT ALIGNED -->
+    <xacro:unless value="${align_depth}">
+      <gazebo reference="${depth_frame}">
+        <self_collide>0</self_collide>
+        <enable_wind>0</enable_wind>
+        <kinematic>0</kinematic>
+        <mu2>1</mu2>
+        <fdir1>0 0 0</fdir1>
+        <kp>1e+13</kp>
+        <kd>1</kd>
+        <sensor name="${camera_name}_depth" type="depth">
+          <topic>${camera_name}/depth/image_raw</topic>
+          <gz_frame_id>${depth_frame}</gz_frame_id>
+          <camera name="${camera_name}_depth_camera">
+            <camera_info_topic>${camera_name}/depth/camera_info</camera_info_topic>
+            <optical_frame_id>${depth_optical_frame}</optical_frame_id>
+            <horizontal_fov>${85.2*deg_to_rad}</horizontal_fov>
+            <image>
+              <width>${depth_width}</width>
+              <height>${depth_height}</height>
+            </image>
+            <clip>
+              <near>${clip_distance_min}</near>
+              <xacro:unless value="${clip_distance > 0.0}">
+                <far>10</far>
+              </xacro:unless>
+              <xacro:if value="${clip_distance > 0.0}">
+                <far>${clip_distance}</far>
+              </xacro:if>
+            </clip>
+            <lens>
               <projection>
                 <p_fx>${depth_fx}</p_fx>
@@ -247,34 +297,12 @@
                 <s>0</s>
               </intrinsics>
-            </xacro:unless>
-            <xacro:if value="${align_depth}">
-              <projection>
-                <p_fx>${color_fx}</p_fx>
-                <p_fy>${color_fy}</p_fy>
-                <p_cx>${color_cx}</p_cx>
-                <p_cy>${color_cy}</p_cy>
-                <tx>0</tx>
-                <ty>0</ty>
-              </projection>
-              <intrinsics>
-                <fx>${color_fx}</fx>
-                <fy>${color_fy}</fy>
-                <cx>${color_cx}</cx>
-                <cy>${color_cy}</cy>
-                <s>0</s>
-              </intrinsics>
-            </xacro:if>
-          </lens>
-        </camera>
-        <always_on>1</always_on>
-        <xacro:unless value="${align_depth}">
+            </lens>
+          </camera>
+          <always_on>1</always_on>
           <update_rate>${depth_fps}</update_rate>
-        </xacro:unless>
-        <xacro:if value="${align_depth}">
-          <update_rate>${color_fps}</update_rate>
-        </xacro:if>
-        <visualize>false</visualize>
-      </sensor>
-    </gazebo>
+          <visualize>false</visualize>
+        </sensor>
+      </gazebo>
+    </xacro:unless>
   </xacro:macro>
 </robot>

File: urdf/_d435.urdf.xacro (robot description, xacro)
@@ -24,4 +24,5 @@
   <xacro:include filename="$(find realsense_gazebo_description)/urdf/_usb_plug.urdf.xacro" />
   <xacro:include filename="$(find realsense_gazebo_description)/urdf/_d435.gazebo.xacro" />
+  <xacro:include filename="$(find realsense_gazebo_description)/urdf/_d435_gazebo_config.xacro" />
   <xacro:macro name="sensor_d435" params="parent
                                           name:=camera
@@ -29,7 +30,7 @@
                                           add_plug:=false
                                           use_mesh:=true
-                                          publish_pointcloud:=false
-                                          align_depth:=true
+                                          align_depth:=false
                                           gazebo_urdf:=false
+                                          custom_intrinsic:=false
                                           clip_distance:=-1.0
                                           clip_distance_min:=0.195
@@ -41,5 +42,5 @@
                                           depth_cx:= 423.82025146484375
                                           depth_cy:= 241.2349395751953
-                                          infra_enable:=false
+                                          enable_infrared:=false
                                           infra_width:=640
                                           infra_height:=480
@@ -61,5 +62,29 @@
     <xacro:property name="M_PI" value="3.1415926535897931" />
     <xacro:property name= "GAZEBO_URDF" value="${gazebo_urdf}" /> <!-- set true to load gazebo plugins -->
-    <xacro:property name="INFRARED" value="${infra_enable}" /> <!-- Set true to enable infrared sensors-->
+    <xacro:property name="INFRARED" value="${enable_infrared}" /> <!-- Set true to enable infrared sensors-->
+    <xacro:d435_gazebo_config custom_intrinsic="${custom_intrinsic}"
+                              clip_distance_min="${clip_distance_min}"
+                              depth_width="${depth_width}"
+                              depth_height="${depth_height}"
+                              depth_fps="${depth_fps}"
+                              depth_fx="${depth_fx}"
+                              depth_fy="${depth_fy}"
+                              depth_cx="${depth_cx}"
+                              depth_cy="${depth_cy}"
+                              infra_width="${infra_width}"
+                              infra_height="${infra_height}"
+                              infra_fps="${infra_fps}"
+                              infra_fx="${infra_fx}"
+                              infra_fy="${infra_fy}"
+                              infra_cx="${infra_cx}"
+                              infra_cy="${infra_cy}"
+                              infra2_tx="${infra2_tx}"
+                              color_width="${color_width}"
+                              color_height="${color_height}"
+                              color_fps="${color_fps}"
+                              color_fx="${color_fx}"
+                              color_fy="${color_fy}"
+                              color_cx="${color_cx}"
+                              color_cy="${color_cy}" />
     <!-- The following values are approximate, and the camera node
      publishing TF values with actual calibrated camera extrinsic values -->
@@ -101,5 +126,6 @@
         <xacro:if value="${use_mesh}">
           <!-- the mesh origin is at front plate in between the two infrared camera axes -->
-          <origin xyz="${d435_zero_depth_to_glass + d435_glass_to_front} ${-d435_cam_depth_py} 0" rpy="${M_PI/2} 0 ${M_PI/2}"/>
+          <!-- <origin xyz="${-d435_zero_depth_to_glass - d435_glass_to_front - 0.006} ${-d435_cam_depth_py} 0" rpy="0 0 ${M_PI/2}"/> -->
+          <origin xyz="${-d435_cam_depth_py - 0.003} ${-d435_cam_depth_py} 0" rpy="0 0 ${M_PI/2}"/>
           <geometry>
             <mesh filename="file://$(find realsense_gazebo_description)/meshes/d435.dae" />
@@ -190,36 +216,39 @@
     <xacro:if value="${GAZEBO_URDF}">
       <!-- Realsense Gazebo Plugin -->
+      <!-- Resolved intrinsic parameters are evaluated in '_d435_gazebo_config.xacro' file -->
       <xacro:gazebo_d435 camera_name="${name}"
-                       reference_link="${name}_link"
+                       color_frame="${name}_color_frame"
+                       depth_frame="${name}_depth_frame"
+                       infrared1_frame="${name}_infra1_frame"
+                       infrared2_frame="${name}_infra2_frame"
                        depth_optical_frame="${name}_depth_optical_frame"
-                       depth_width="${depth_width}"
-                       depth_height="${depth_height}"
-                       depth_fps="${depth_fps}"
-                       depth_fx="${depth_fx}"
-                       depth_fy="${depth_fy}"
-                       depth_cx="${depth_cx}"
-                       depth_cy="${depth_cy}"
+                       depth_width="${resolved_depth_width}"
+                       depth_height="${resolved_depth_height}"
+                       depth_fps="${resolved_depth_fps}"
+                       depth_fx="${resolved_depth_fx}"
+                       depth_fy="${resolved_depth_fy}"
+                       depth_cx="${resolved_depth_cx}"
+                       depth_cy="${resolved_depth_cy}"
                        color_optical_frame="${name}_color_optical_frame"
-                       color_width="${color_width}"
-                       color_height="${color_height}"
-                       color_fps="${color_fps}"
-                       color_fx="${color_fx}"
-                       color_fy="${color_fy}"
-                       color_cx="${color_cx}"
-                       color_cy="${color_cy}"
-                       infrared1_optical_frame="${name}_infra1_ir_optical_frame"
-                       infrared2_optical_frame="${name}_infra2_ir_optical_frame"
-                       infra_enable="${infra_enable}"
-                       infra_width="${infra_width}"
-                       infra_height="${infra_height}"
-                       infra_fps="${infra_fps}"
-                       infra_fx="${infra_fx}"
-                       infra_fy="${infra_fy}"
-                       infra_cx="${infra_cx}"
-                       infra_cy="${infra_cy}"
-                       infra2_tx="${infra2_tx}"
-                       publish_pointcloud="${publish_pointcloud}"
+                       color_width="${resolved_color_width}"
+                       color_height="${resolved_color_height}"
+                       color_fps="${resolved_color_fps}"
+                       color_fx="${resolved_color_fx}"
+                       color_fy="${resolved_color_fy}"
+                       color_cx="${resolved_color_cx}"
+                       color_cy="${resolved_color_cy}"
+                       infrared1_optical_frame="${name}_infra1_optical_frame"
+                       infrared2_optical_frame="${name}_infra2_optical_frame"
+                       enable_infrared="${enable_infrared}"
+                       infra_width="${resolved_infra_width}"
+                       infra_height="${resolved_infra_height}"
+                       infra_fps="${resolved_infra_fps}"
+                       infra_fx="${resolved_infra_fx}"
+                       infra_fy="${resolved_infra_fy}"
+                       infra_cx="${resolved_infra_cx}"
+                       infra_cy="${resolved_infra_cy}"
+                       infra2_tx="${resolved_infra2_tx}"
                        clip_distance="${clip_distance}"
-                       clip_distance_min="${clip_distance_min}"
+                       clip_distance_min="${resolved_clip_distance_min}"
                        align_depth="${align_depth}"
                        visualize="${visualize}"
