Commit message: Added adaptive intrinsic based on image resolution like in the real camera
Updated mesh and material to visualize the model properly

File: urdf/_d435_gazebo_config.xacro (robot description, xacro)
@@ -1,98 +1,166 @@
 <?xml version="1.0"?>
 <robot xmlns:xacro="http://ros.org/wiki/xacro" name="sensor_d435_gazebo_config">
-<!-- Actually confid file not in use to not disrupt all the macros
- that all the various robot are using. But kept for reference for different res/parameters -->
-<!-- Taken from real camera, official realsenselib for ros Noetic -->
-<xacro:arg name="color_res" default="640x480"/>
-<xacro:property name="COLOR_RES" value="$(arg color_res)" />
-<xacro:arg name="depth_res" default="848x480"/>
-<xacro:property name="DEPTH_RES" value="$(arg depth_res)" />
-<xacro:arg name="infra_res" default="640x480"/>
-<xacro:property name="INFRA_RES" value="$(arg infra_res)" />
-<xacro:if value="${COLOR_RES == '1920x1080'}">
-  <xacro:property name="color_width" value="1920"/>
-  <xacro:property name="color_height" value="1080"/>
-  <xacro:property name="color_fps" value="30"/> <!--6 15 30-->
-  <xacro:property name="color_fx" value="1364.58154296875"/>
-  <xacro:property name="color_fy" value="1364.4825439453125"/>
-  <xacro:property name="color_cx" value="974.0638427734375"/>
-  <xacro:property name="color_cy" value="572.7390747070312"/>
-</xacro:if>
-<xacro:if value="${COLOR_RES == '1280x720'}">
-  <xacro:property name="color_width" value="1280"/>
-  <xacro:property name="color_height" value="720"/>
-  <xacro:property name="color_fps" value="30"/> <!--6 15 30-->
-  <xacro:property name="color_fx" value="909.7210083007812"/>
-  <xacro:property name="color_fy" value="909.655029296875"/>
-  <xacro:property name="color_cx" value="649.3759155273438"/>
-  <xacro:property name="color_cy" value="381.8260498046875"/>
-</xacro:if>
-<xacro:if value="${COLOR_RES == '960x540'}"></xacro:if>
-<xacro:if value="${COLOR_RES == '848x480'}"></xacro:if>
-<xacro:if value="${COLOR_RES == '640x480'}"> <!--default roslaunch of real cam-->
-  <xacro:property name="color_width" value="640"/>
-  <xacro:property name="color_height" value="480"/>
-  <xacro:property name="color_fps" value="30"/> <!--6 15 30 60-->
-  <xacro:property name="color_fx" value="606.4806518554688"/>
-  <xacro:property name="color_fy" value="606.4366455078125"/>
-  <xacro:property name="color_cx" value="326.2506103515625"/>
-  <xacro:property name="color_cy" value="254.5507049560547"/>
-</xacro:if>
-<xacro:if value="${COLOR_RES == '640x360'}"></xacro:if>
-<xacro:if value="${COLOR_RES == '424x240'}"></xacro:if>
-<xacro:if value="${COLOR_RES == '320x240'}"></xacro:if>
-<xacro:if value="${COLOR_RES == '320x180'}"></xacro:if>
-<!-- NOTE: on real camera, for the aligned to color version the instrisic are the same of color one -->
-<xacro:if value="${DEPTH_RES == '1280x720'}">
-  <xacro:property name="depth_width" value="1280"/>
-  <xacro:property name="depth_height" value="720"/>
-  <xacro:property name="depth_fps" value="30"/> <!--  6 15 30 for this res -->
-  <xacro:property name="depth_fx" value="650.98046875"/>
-  <xacro:property name="depth_fy" value="650.98046875"/>
-  <xacro:property name="depth_cx" value="639.7286987304688"/>
-  <xacro:property name="depth_cy" value="361.9244384765625"/>
-  <xacro:property name="clip_distance_min" value="0.280"/>
-</xacro:if>
-<xacro:if value="${DEPTH_RES == '848x480'}"> <!--default roslaunch of real cam-->
-  <xacro:property name="depth_width" value="848"/>
-  <xacro:property name="depth_height" value="480"/>
-  <xacro:property name="depth_fps" value="30"/> <!-- 6 15 30 60 90 avaiable from this to lower res -->
-  <xacro:property name="depth_fx" value="431.2745666503906"/>
-  <xacro:property name="depth_fy" value="431.2745666503906"/>
-  <xacro:property name="depth_cx" value="423.82025146484375"/>
-  <xacro:property name="depth_cy" value="241.2349395751953"/>
-  <xacro:property name="clip_distance_min" value="0.195"/>
-</xacro:if>
-<xacro:if value="${DEPTH_RES == '640x480'}">
-  <xacro:property name="depth_width" value="640"/>
-  <xacro:property name="depth_height" value="480"/>
-  <xacro:property name="depth_fps" value="30"/> <!-- 6 15 30 60 90 avaiable from this to lower res -->
-  <xacro:property name="depth_fx" value="390.5882873535156"/>
-  <xacro:property name="depth_fy" value="390.5882873535156"/>
-  <xacro:property name="depth_cx" value="319.83721923828125"/>
-  <xacro:property name="depth_cy" value="241.14466857910156"/>
-  <xacro:property name="clip_distance_min" value="0.175"/>
-</xacro:if>
-<xacro:if value="${DEPTH_RES == '640x360'}"></xacro:if>
-<xacro:if value="${DEPTH_RES == '480x270'}"></xacro:if>
-<xacro:if value="${DEPTH_RES == '424x240'}">
-  <xacro:property name="depth_width" value="424"/>
-  <xacro:property name="depth_height" value="240"/>
-  <xacro:property name="depth_fps" value="30"/>
-  <xacro:property name="depth_fx" value="215.6372833251953"/>
-  <xacro:property name="depth_fy" value="215.6372833251953"/>
-  <xacro:property name="depth_cx" value="211.91012573242188"/>
-  <xacro:property name="depth_cy" value="120.63746643066406"/>
-  <xacro:property name="clip_distance_min" value="0.105"/>
-</xacro:if>
-<xacro:if value="${INFRA_RES == '640x480'}">
-  <xacro:property name="infra_width" value="640"/>
-  <xacro:property name="infra_height" value="480"/>
-  <xacro:property name="infra_fps" value="30"/>
-  <xacro:property name="infra_fx" value="431.2745666503906"/>
-  <xacro:property name="infra_fy" value="431.2745666503906"/>
-  <xacro:property name="infra_cx" value="423.82025146484375"/>
-  <xacro:property name="infra_cy" value="241.2349395751953"/>
-  <xacro:property name="infra2_tx" value="-21.57023811340332"/>
-</xacro:if>
+  <!-- Taken from real camera, official realsenselib for ros Noetic -->
+  <!-- Resolve the effective camera parameters from either the user-provided
+       intrinsics or the known intrinsics associated with the selected image
+       resolution. -->
+  <xacro:macro name="d435_gazebo_config" params="
+                                            custom_intrinsic:=false
+                                            clip_distance_min:=0.195
+                                            depth_width:=848
+                                            depth_height:=480
+                                            depth_fps:=30
+                                            depth_fx:=431.2745666503906
+                                            depth_fy:=431.2745666503906
+                                            depth_cx:=423.82025146484375
+                                            depth_cy:=241.2349395751953
+                                            infra_width:=640
+                                            infra_height:=480
+                                            infra_fps:=30
+                                            infra_fx:=431.2745666503906
+                                            infra_fy:=431.2745666503906
+                                            infra_cx:=423.82025146484375
+                                            infra_cy:=241.2349395751953
+                                            infra2_tx:=-21.57023811340332
+                                            color_width:=640
+                                            color_height:=480
+                                            color_fps:=30
+                                            color_fx:=606.4806518554688
+                                            color_fy:=606.4366455078125
+                                            color_cx:=326.2506103515625
+                                            color_cy:=254.5507049560547">
+    <xacro:property name="resolved_clip_distance_min" value="${clip_distance_min}" scope="parent" />
+    <xacro:property name="resolved_depth_width" value="${depth_width}" scope="parent" />
+    <xacro:property name="resolved_depth_height" value="${depth_height}" scope="parent" />
+    <xacro:property name="resolved_depth_fps" value="${depth_fps}" scope="parent" />
+    <xacro:property name="resolved_depth_fx" value="${depth_fx}" scope="parent" />
+    <xacro:property name="resolved_depth_fy" value="${depth_fy}" scope="parent" />
+    <xacro:property name="resolved_depth_cx" value="${depth_cx}" scope="parent" />
+    <xacro:property name="resolved_depth_cy" value="${depth_cy}" scope="parent" />
+    <xacro:property name="resolved_infra_width" value="${infra_width}" scope="parent" />
+    <xacro:property name="resolved_infra_height" value="${infra_height}" scope="parent" />
+    <xacro:property name="resolved_infra_fps" value="${infra_fps}" scope="parent" />
+    <xacro:property name="resolved_infra_fx" value="${infra_fx}" scope="parent" />
+    <xacro:property name="resolved_infra_fy" value="${infra_fy}" scope="parent" />
+    <xacro:property name="resolved_infra_cx" value="${infra_cx}" scope="parent" />
+    <xacro:property name="resolved_infra_cy" value="${infra_cy}" scope="parent" />
+    <xacro:property name="resolved_infra2_tx" value="${infra2_tx}" scope="parent" />
+    <xacro:property name="resolved_color_width" value="${color_width}" scope="parent" />
+    <xacro:property name="resolved_color_height" value="${color_height}" scope="parent" />
+    <xacro:property name="resolved_color_fps" value="${color_fps}" scope="parent" />
+    <xacro:property name="resolved_color_fx" value="${color_fx}" scope="parent" />
+    <xacro:property name="resolved_color_fy" value="${color_fy}" scope="parent" />
+    <xacro:property name="resolved_color_cx" value="${color_cx}" scope="parent" />
+    <xacro:property name="resolved_color_cy" value="${color_cy}" scope="parent" />
+    <xacro:unless value="${custom_intrinsic}">
+      <xacro:property name="COLOR_RES" value="${str(color_width) + 'x' + str(color_height)}" />
+      <xacro:property name="DEPTH_RES" value="${str(depth_width) + 'x' + str(depth_height)}" />
+      <xacro:property name="INFRA_RES" value="${str(infra_width) + 'x' + str(infra_height)}" />
+      <!-- COLOR INTRINSICS -->
+      <xacro:if value="${COLOR_RES == '1920x1080'}">
+        <xacro:property name="resolved_color_width" value="1920" scope="parent" />
+        <xacro:property name="resolved_color_height" value="1080" scope="parent" />
+        <xacro:property name="resolved_color_fps" value="30" scope="parent" /> <!--6 15 30-->
+        <xacro:property name="resolved_color_fx" value="1364.58154296875" scope="parent" />
+        <xacro:property name="resolved_color_fy" value="1364.4825439453125" scope="parent" />
+        <xacro:property name="resolved_color_cx" value="974.0638427734375" scope="parent" />
+        <xacro:property name="resolved_color_cy" value="572.7390747070312" scope="parent" />
+      </xacro:if>
+      <xacro:if value="${COLOR_RES == '1280x720'}">
+        <xacro:property name="resolved_color_width" value="1280" scope="parent" />
+        <xacro:property name="resolved_color_height" value="720" scope="parent" />
+        <xacro:property name="resolved_color_fps" value="30" scope="parent" /> <!--6 15 30-->
+        <xacro:property name="resolved_color_fx" value="909.7210083007812" scope="parent" />
+        <xacro:property name="resolved_color_fy" value="909.655029296875" scope="parent" />
+        <xacro:property name="resolved_color_cx" value="649.3759155273438" scope="parent" />
+        <xacro:property name="resolved_color_cy" value="381.8260498046875" scope="parent" />
+      </xacro:if>
+      <xacro:if value="${COLOR_RES == '640x480'}">
+        <xacro:property name="resolved_color_width" value="640" scope="parent" />
+        <xacro:property name="resolved_color_height" value="480" scope="parent" />
+        <xacro:property name="resolved_color_fps" value="30" scope="parent" /> <!--6 15 30 60-->
+        <xacro:property name="resolved_color_fx" value="606.4806518554688" scope="parent" />
+        <xacro:property name="resolved_color_fy" value="606.4366455078125" scope="parent" />
+        <xacro:property name="resolved_color_cx" value="326.2506103515625" scope="parent" />
+        <xacro:property name="resolved_color_cy" value="254.5507049560547" scope="parent" />
+      </xacro:if>
+      <xacro:if value="${COLOR_RES == '640x480'}">
+        <xacro:property name="resolved_color_width" value="640" scope="parent" />
+        <xacro:property name="resolved_color_height" value="480" scope="parent" />
+        <xacro:property name="resolved_color_fps" value="30" scope="parent" /> <!--6 15 30 60-->
+        <xacro:property name="resolved_color_fx" value="606.4806518554688" scope="parent" />
+        <xacro:property name="resolved_color_fy" value="606.4366455078125" scope="parent" />
+        <xacro:property name="resolved_color_cx" value="326.2506103515625" scope="parent" />
+        <xacro:property name="resolved_color_cy" value="254.5507049560547" scope="parent" />
+      </xacro:if><xacro:if value="${COLOR_RES == '640x480'}">
+        <xacro:property name="resolved_color_width" value="640" scope="parent" />
+        <xacro:property name="resolved_color_height" value="480" scope="parent" />
+        <xacro:property name="resolved_color_fps" value="30" scope="parent" /> <!--6 15 30 60-->
+        <xacro:property name="resolved_color_fx" value="606.4806518554688" scope="parent" />
+        <xacro:property name="resolved_color_fy" value="606.4366455078125" scope="parent" />
+        <xacro:property name="resolved_color_cx" value="326.2506103515625" scope="parent" />
+        <xacro:property name="resolved_color_cy" value="254.5507049560547" scope="parent" />
+      </xacro:if>
+      <xacro:if value="${COLOR_RES == '640x480'}">
+        <xacro:property name="resolved_color_width" value="640" scope="parent" />
+        <xacro:property name="resolved_color_height" value="480" scope="parent" />
+        <xacro:property name="resolved_color_fps" value="30" scope="parent" /> <!--6 15 30 60-->
+        <xacro:property name="resolved_color_fx" value="606.4806518554688" scope="parent" />
+        <xacro:property name="resolved_color_fy" value="606.4366455078125" scope="parent" />
+        <xacro:property name="resolved_color_cx" value="326.2506103515625" scope="parent" />
+        <xacro:property name="resolved_color_cy" value="254.5507049560547" scope="parent" />
+      </xacro:if>
+      <xacro:if value="${COLOR_RES == '640x480'}">
+        <xacro:property name="resolved_color_width" value="640" scope="parent" />
+        <xacro:property name="resolved_color_height" value="480" scope="parent" />
+        <xacro:property name="resolved_color_fps" value="30" scope="parent" /> <!--6 15 30 60-->
+        <xacro:property name="resolved_color_fx" value="606.4806518554688" scope="parent" />
+        <xacro:property name="resolved_color_fy" value="606.4366455078125" scope="parent" />
+        <xacro:property name="resolved_color_cx" value="326.2506103515625" scope="parent" />
+        <xacro:property name="resolved_color_cy" value="254.5507049560547" scope="parent" />
+      </xacro:if>
+      <!-- DEPTH INTRINSICS -->
+      <xacro:if value="${DEPTH_RES == '1280x720'}">
+        <xacro:property name="resolved_depth_width" value="1280" scope="parent" />
+        <xacro:property name="resolved_depth_height" value="720" scope="parent" />
+        <xacro:property name="resolved_depth_fps" value="30" scope="parent" />
+        <xacro:property name="resolved_depth_fx" value="650.98046875" scope="parent" />
+        <xacro:property name="resolved_depth_fy" value="650.98046875" scope="parent" />
+        <xacro:property name="resolved_depth_cx" value="639.7286987304688" scope="parent" />
+        <xacro:property name="resolved_depth_cy" value="361.9244384765625" scope="parent" />
+        <xacro:property name="resolved_clip_distance_min" value="0.280" scope="parent" />
+      </xacro:if>
+      <xacro:if value="${DEPTH_RES == '848x480'}">
+        <xacro:property name="resolved_depth_width" value="848" scope="parent" />
+        <xacro:property name="resolved_depth_height" value="480" scope="parent" />
+        <xacro:property name="resolved_depth_fps" value="30" scope="parent" />
+        <xacro:property name="resolved_depth_fx" value="431.2745666503906" scope="parent" />
+        <xacro:property name="resolved_depth_fy" value="431.2745666503906" scope="parent" />
+        <xacro:property name="resolved_depth_cx" value="423.82025146484375" scope="parent" />
+        <xacro:property name="resolved_depth_cy" value="241.2349395751953" scope="parent" />
+        <xacro:property name="resolved_clip_distance_min" value="0.195" scope="parent" />
+      </xacro:if>
+      <xacro:if value="${DEPTH_RES == '640x480'}">
+        <xacro:property name="resolved_depth_width" value="640" scope="parent" />
+        <xacro:property name="resolved_depth_height" value="480" scope="parent" />
+        <xacro:property name="resolved_depth_fps" value="30" scope="parent" />
+        <xacro:property name="resolved_depth_fx" value="390.5882873535156" scope="parent" />
+        <xacro:property name="resolved_depth_fy" value="390.5882873535156" scope="parent" />
+        <xacro:property name="resolved_depth_cx" value="319.83721923828125" scope="parent" />
+        <xacro:property name="resolved_depth_cy" value="241.14466857910156" scope="parent" />
+        <xacro:property name="resolved_clip_distance_min" value="0.175" scope="parent" />
+      </xacro:if>
+      <!-- INFRARED INTRINSICS -->
+      <xacro:if value="${INFRA_RES == '640x480'}">
+        <xacro:property name="resolved_infra_width" value="640" scope="parent" />
+        <xacro:property name="resolved_infra_height" value="480" scope="parent" />
+        <xacro:property name="resolved_infra_fps" value="30" scope="parent" />
+        <xacro:property name="resolved_infra_fx" value="431.2745666503906" scope="parent" />
+        <xacro:property name="resolved_infra_fy" value="431.2745666503906" scope="parent" />
+        <xacro:property name="resolved_infra_cx" value="423.82025146484375" scope="parent" />
+        <xacro:property name="resolved_infra_cy" value="241.2349395751953" scope="parent" />
+        <xacro:property name="resolved_infra2_tx" value="-21.57023811340332" scope="parent" />
+      </xacro:if>
+    </xacro:unless>
+  </xacro:macro>
 </robot>

File: urdf/d435_standalone.urdf.xacro (robot description, xacro)
@@ -10,9 +10,10 @@
     <xacro:arg name="yaw" default="0"/>
     <xacro:arg name="align_depth" default="false"/>
+    <xacro:arg name="custom_intrinsic" default="false"/>
     <xacro:arg name="use_nominal_extrinsics" default="false"/>
     <xacro:arg name="add_plug" default="false" />
     <xacro:arg name="use_mesh" default="true" />
     <xacro:arg name="gazebo_urdf" default="false" />
-    <xacro:arg name="infra_enable" default="false"/>
+    <xacro:arg name="enable_infrared" default="false"/>
 	<xacro:include filename="$(find realsense_gazebo_description)/urdf/_d435.urdf.xacro"/>
  	<link name="$(arg parent)"/>
@@ -20,5 +21,6 @@
         use_nominal_extrinsics="$(arg use_nominal_extrinsics)" add_plug="$(arg add_plug)"
         use_mesh="$(arg use_mesh)" gazebo_urdf="$(arg gazebo_urdf)"
-        infra_enable="$(arg infra_enable)" align_depth="$(arg align_depth)">
+        enable_infrared="$(arg enable_infrared)" align_depth="$(arg align_depth)"
+        custom_intrinsic="$(arg custom_intrinsic)">
 		<origin xyz="$(arg x) $(arg y) $(arg z)" rpy="$(arg roll) $(arg pitch) $(arg yaw)"/>
 	</xacro:sensor_d435>
