Commit message: correct package name

File: urdf/_d435.urdf.xacro (robot description, xacro)
@@ -100,5 +100,5 @@
           <origin xyz="${d435_zero_depth_to_glass + d435_glass_to_front} ${-d435_cam_depth_py} 0" rpy="${M_PI/2} 0 ${M_PI/2}"/>
           <geometry>
-            <mesh filename="file://$(find realsense2_description)/meshes/d435.dae" />
+            <mesh filename="file://$(find realsense_gazebo_description)/meshes/d435.dae" />
           </geometry>
         </xacro:if>
@@ -106,5 +106,5 @@
           <origin xyz="${d435_zero_depth_to_glass + d435_glass_to_front} ${-d435_cam_depth_py} 0" rpy="${M_PI/2} 0 ${M_PI/2}"/>
           <geometry>
-            <mesh filename="file://$(find realsense2_description)/meshes/d435_simplified.stl" />
+            <mesh filename="file://$(find realsense_gazebo_description)/meshes/d435_simplified.stl" />
           </geometry>
           <material name="aluminum"/>

Commit message: Reverted xacro files to match 'realsense2_description' package and updated rviz default file's name in launch file. No gazebo integration yet.

File: urdf/_d435.urdf.xacro (robot description, xacro)
@@ -23,5 +23,4 @@
   <xacro:include filename="$(find realsense_gazebo_description)/urdf/_materials.urdf.xacro" />
   <xacro:include filename="$(find realsense_gazebo_description)/urdf/_usb_plug.urdf.xacro" />
-  <xacro:include filename="$(find realsense_gazebo_description)/urdf/_d435.gazebo.xacro" />
   <xacro:macro name="sensor_d435" params="parent
                                           name:=camera
@@ -182,39 +181,4 @@
       </xacro:usb_plug>
     </xacro:if>
-    <!-- Realsense Gazebo Plugin -->
-    <xacro:gazebo_d435 camera_name="${name}"
-                       reference_link="${name}_link"
-                       depth_optical_frame="${name}_depth_optical_frame"
-                       depth_width="${depth_width}"
-                       depth_height="${depth_height}"
-                       depth_fps="${depth_fps}"
-                       depth_fx="${depth_fx}"
-                       depth_fy="${depth_fy}"
-                       depth_cx="${depth_cx}"
-                       depth_cy="${depth_cy}"
-                       color_optical_frame="${name}_color_optical_frame"
-                       color_width="${color_width}"
-                       color_height="${color_height}"
-                       color_fps="${color_fps}"
-                       color_fx="${color_fx}"
-                       color_fy="${color_fy}"
-                       color_cx="${color_cx}"
-                       color_cy="${color_cy}"
-                       infrared1_optical_frame="${name}_infra1_ir_optical_frame"
-                       infrared2_optical_frame="${name}_infra2_ir_optical_frame"
-                       infra_width="${infra_width}"
-                       infra_height="${infra_height}"
-                       infra_fps="${infra_fps}"
-                       infra_fx="${infra_fx}"
-                       infra_fy="${infra_fy}"
-                       infra_cx="${infra_cx}"
-                       infra_cy="${infra_cy}"
-                       infra2_tx="${infra2_tx}"
-                       publish_pointcloud="${publish_pointcloud}"
-                       clip_distance="${clip_distance}"
-                       clip_distance_min="${clip_distance_min}"
-                       align_depth="${align_depth}"
-                       visualize="${visualize}"
-    />
   </xacro:macro>
 </robot>

File: urdf/_d435i.urdf.xacro (robot description, xacro)
@@ -23,5 +23,4 @@
   <xacro:include filename="$(find realsense_gazebo_description)/urdf/_materials.urdf.xacro" />
   <xacro:include filename="$(find realsense_gazebo_description)/urdf/_usb_plug.urdf.xacro" />
-  <xacro:include filename="$(find realsense_gazebo_description)/urdf/_d435i.gazebo.xacro" />
   <xacro:macro name="sensor_d435i" params="parent
                                           name:=camera
@@ -56,7 +55,4 @@
                                           color_cy:= 254.5507049560547
                                           visualize:=false
-                                          unite_imu_method:=false
-                                          accel_fps:=250
-                                          gyro_fps:=400
                                           *origin">
     <xacro:property name="M_PI" value="3.1415926535897931" />
@@ -180,29 +176,29 @@
       <link name="${name}_color_optical_frame"/>
       <!-- camera accel joints and links -->
+      <link name="${name}_accel_frame" />
       <joint name="${name}_accel_joint" type="fixed">
-        <origin xyz="-0.00174 0.00552 0.0176" rpy="0 0 0"/>
-        <parent link="${name}_link"/>
-        <child link="${name}_accel_frame"/>
-      </joint>
-      <link name="${name}_accel_frame"/>
+        <origin xyz = "-0.01174 -0.00552 0.0051" rpy = "0 0 0" />
+        <parent link="${name}_link" />
+        <child link="${name}_accel_frame" />
+      </joint>
+      <link name="${name}_accel_optical_frame"/>
       <joint name="${name}_accel_optical_joint" type="fixed">
-        <origin xyz="0 0 0" rpy="${-M_PI/2} 0 ${-M_PI/2}"/>
-        <parent link="${name}_accel_frame"/>
-        <child link="${name}_accel_optical_frame"/>
-      </joint>
-      <link name="${name}_accel_optical_frame"/>
+        <origin xyz = "0 0 0" rpy = "${-M_PI/2} 0 ${-M_PI/2}" />
+        <parent link="${name}_accel_frame" />
+        <child link="${name}_accel_optical_frame" />
+      </joint>
       <!-- camera gyro joints and links -->
+      <link name="${name}_gyro_frame"/>
       <joint name="${name}_gyro_joint" type="fixed">
-        <origin xyz="-0.00174 0.00552 0.0176" rpy="0 0 0"/>
-        <parent link="${name}_link"/>
-        <child link="${name}_gyro_frame"/>
-      </joint>
-      <link name="${name}_gyro_frame"/>
+        <origin xyz = "-0.01174 -0.00552 0.0051" rpy = "0 0 0" />
+        <parent link="${name}_link" />
+        <child link="${name}_gyro_frame" />
+      </joint>
+      <link name="${name}_gyro_optical_frame"/>
       <joint name="${name}_gyro_optical_joint" type="fixed">
-        <origin xyz="0 0 0" rpy="${-M_PI/2} 0 ${-M_PI/2}"/>
-        <parent link="${name}_gyro_frame"/>
-        <child link="${name}_gyro_optical_frame"/>
-      </joint>
-      <link name="${name}_gyro_optical_frame"/>
+        <origin xyz = "0 0 0" rpy = "${-M_PI/2} 0 ${-M_PI/2}" />
+        <parent link="${name}_gyro_frame" />
+        <child link="${name}_gyro_optical_frame" />
+      </joint>
     </xacro:if>
     <xacro:if value="${add_plug}">
@@ -211,44 +207,4 @@
       </xacro:usb_plug>
     </xacro:if>
-    <!-- Realsense Gazebo Plugin -->
-    <xacro:gazebo_d435i camera_name="${name}"
-                       reference_link="${name}_link"
-                       depth_optical_frame="${name}_depth_optical_frame"
-                       depth_width="${depth_width}"
-                       depth_height="${depth_height}"
-                       depth_fps="${depth_fps}"
-                       depth_fx="${depth_fx}"
-                       depth_fy="${depth_fy}"
-                       depth_cx="${depth_cx}"
-                       depth_cy="${depth_cy}"
-                       color_optical_frame="${name}_color_optical_frame"
-                       color_width="${color_width}"
-                       color_height="${color_height}"
-                       color_fps="${color_fps}"
-                       color_fx="${color_fx}"
-                       color_fy="${color_fy}"
-                       color_cx="${color_cx}"
-                       color_cy="${color_cy}"
-                       infrared1_optical_frame="${name}_infra1_ir_optical_frame"
-                       infrared2_optical_frame="${name}_infra2_ir_optical_frame"
-                       infra_width="${infra_width}"
-                       infra_height="${infra_height}"
-                       infra_fps="${infra_fps}"
-                       infra_fx="${infra_fx}"
-                       infra_fy="${infra_fy}"
-                       infra_cx="${infra_cx}"
-                       infra_cy="${infra_cy}"
-                       infra2_tx="${infra2_tx}"
-                       publish_pointcloud="${publish_pointcloud}"
-                       clip_distance="${clip_distance}"
-                       clip_distance_min="${clip_distance_min}"
-                       align_depth="${align_depth}"
-                       visualize="${visualize}"
-                        accel_optical_frame="${name}_accel_optical_frame"
-                        gyro_optical_frame="${name}_gyro_optical_frame"
-                        accel_fps="${accel_fps}"
-                        gyro_fps="${gyro_fps}"
-                        unite_imu_method="${unite_imu_method}"
-    />
   </xacro:macro>
 </robot>

File: urdf/d435_standalone.urdf.xacro (robot description, xacro)
@@ -11,7 +11,12 @@
     <xacro:arg name="publish_pointcloud" default="false"/>
     <xacro:arg name="align_depth" default="false"/>
+    <xacro:arg name="use_nominal_extrinsics" default="false"/>
+    <xacro:arg name="add_plug" default="false" />
+    <xacro:arg name="use_mesh" default="true" />
 	<xacro:include filename="$(find realsense_gazebo_description)/urdf/_d435.urdf.xacro"/>
  	<link name="$(arg parent)"/>
-	<xacro:sensor_d435 parent="$(arg parent)" name="$(arg name)" topics_ns="$(arg name)"
+	<xacro:sensor_d435 parent="$(arg parent)" name="$(arg name)"
+        use_nominal_extrinsics="$(arg use_nominal_extrinsics)" add_plug="$(arg add_plug)"
+        use_mesh="$(arg use_mesh)"
         publish_pointcloud="$(arg publish_pointcloud)" align_depth="$(arg align_depth)">
 		<origin xyz="$(arg x) $(arg y) $(arg z)" rpy="$(arg roll) $(arg pitch) $(arg yaw)"/>

File: urdf/d435i_standalone.urdf.xacro (robot description, xacro)
@@ -11,7 +11,12 @@
     <xacro:arg name="publish_pointcloud" default="false"/>
     <xacro:arg name="align_depth" default="false"/>
+    <xacro:arg name="use_nominal_extrinsics" default="false"/>
+    <xacro:arg name="add_plug" default="false" />
+    <xacro:arg name="use_mesh" default="true" />
 	<xacro:include filename="$(find realsense_gazebo_description)/urdf/_d435i.urdf.xacro"/>
  	<link name="$(arg parent)"/>
-	<xacro:sensor_d435i parent="$(arg parent)" name="$(arg name)" topics_ns="$(arg name)"
+	<xacro:sensor_d435i parent="$(arg parent)" name="$(arg name)"
+        use_nominal_extrinsics="$(arg use_nominal_extrinsics)" add_plug="$(arg add_plug)"
+        use_mesh="$(arg use_mesh)"
         publish_pointcloud="$(arg publish_pointcloud)" align_depth="$(arg align_depth)">
 		<origin xyz="$(arg x) $(arg y) $(arg z)" rpy="$(arg roll) $(arg pitch) $(arg yaw)"/>
